File: relays.sch (EAGLE design)
At the start: 45 parts, among them Q1 MMBT2222A, Q2 MMBT2222A, T1 BTA12-600, T2 BTA12-600

Commit message: add some silkscreen
Parts:
- OK3: value MOC3020 -> H11AA1
Changed lines of the file:
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@@
 <part name="OK1" library="optocoupler" deviceset="MOC30*" device="S" technology="31" value="MOC3020"/>
 <part name="U$1" library="SparkFun-Electromechanical" deviceset="RELAY" device="PTH"/>
-<part name="OK3" library="optocoupler" deviceset="H11A*?M" device="S" technology="1" value="MOC3020"/>
+<part name="OK3" library="optocoupler" deviceset="H11A*?M" device="S" technology="1" value="H11AA1"/>
 <part name="GND1" library="SparkFun-Aesthetics" deviceset="GND" device=""/>
 <part name="R1" library="SparkFun-Passives" deviceset="RESISTOR" device="0603-RES" value="1k"/>

Commit message: update relay board, REx. Good boy.
Parts:
- renumbered U$1 to RELAY0, U$2 to RELAY1
Connections:
- net SSD0-HOT renamed SSR0-HOT
- net SSD1-HOT renamed SSR1-HOT
